File: PCB/Zicada Board/Zicada.kicad_sch (KiCad schematic)
At the start: 57 parts, among them J1 Conn_ARM_JTAG_SWD_10, J2 Conn_01x01_Pin, J3 Conn_01x01_Pin, SW1 SW_Push, U1 nRF52840, U2 HDC2080, U3 SM351LT, U4 TPS610981, U5 OPT3001, Y1 32MHz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

Commit message: Everything 0402, 4 layer board
Parts:
- added C101: 100n,16V, Passives:C0402, symbol Device:C
- C1, C4: footprint Capacitor_SMD:C_0603_1608Metric -> Passives:C0402
- C10, C13, C14, C16, C19, C20, C21, C22, C24: value 100nF -> 100n,16V; footprint Capacitor_SMD:C_0603_1608Metric -> Passives:C0402; LCSC C1591 -> (none)
- C11: value 4.7uF -> 10u,6.3V; LCSC C1705 -> (none)
- C12, C2: value 1uF -> 1u,10V; footprint Capacitor_SMD:C_0603_1608Metric -> Passives:C0402; LCSC C15849 -> (none)
- C15, C17, C5, C6: value 12pF -> 12p,50V; footprint Capacitor_SMD:C_0603_1608Metric -> Passives:C0402; LCSC C107034 -> (none)
- C18, C23: value 10uF -> 10u,6.3V; LCSC C19702 -> (none)
- C3: value 820pF -> 820p,50V; footprint Capacitor_SMD:C_0603_1608Metric -> Passives:C0402; LCSC C107057 -> (none)
- C7: value 0.5pF -> 0.5p,50V; footprint Capacitor_SMD:C_0603_1608Metric -> Passives:C0402; LCSC C5137584 -> (none)
- C8: value 100pF -> 100p,50V; footprint Capacitor_SMD:C_0603_1608Metric -> Passives:C0402; LCSC C14858 -> (none)
- C9: value 0.8pF -> 0.8p,50V; footprint Capacitor_SMD:C_0603_1608Metric -> Passives:C0402; LCSC C519369 -> (none)
- FID1, FID2, FID3, FID4: footprint Fiducial:Fiducial_1mm_Mask2mm -> Mechanical:FIDUCIAL_1mm
- J1: footprint Connector_PinHeader_1.27mm:PinHeader_2x05_P1.27mm_Vertical_SMD -> Connector:TC2050-IDC-NLFP
- L1: footprint Inductor_SMD:L_0603_1608Metric -> Passives:L0402; LCSC C1030 -> (none)
- R1, R7: footprint Resistor_SMD:R_0603_1608Metric -> Passives:R0402; LCSC C116699 -> (none)
- R2, R8: footprint Resistor_SMD:R_0603_1608Metric -> Passives:R0402; LCSC C105881 -> (none)
- R3: footprint Resistor_SMD:R_0603_1608Metric -> Passives:R0402; LCSC C105578 -> (none)
- R5, R6: footprint Resistor_SMD:R_0603_1608Metric -> Passives:R0402; LCSC C98220 -> (none)
Connections:
- net GND: now also C101.2
- net VDD: now also C101.1
Other:
- moved on the sheet: C11, C13, C14, C16, C2, C3, C8

Commit message: Add BME688
Parts:
- added C904: 100n,16V, Passives:C0402, symbol Passives:C
- added IC901: BME680, IC:BME680, symbol Sensors:BME680
Connections:
- net GND: now also C904.2, IC901.1 (GND), IC901.7 (GND)
- net SCL: now also IC901.4 (SCK)
- net SDA: now also IC901.3 (SDI)
- net VDD: now also C904.1, IC901.2 (CSB), IC901.5 (SDO), IC901.6 (VDDIO), IC901.8 (VDD)
