File: PCB/Zicada Board/Zicada.kicad_sch (KiCad schematic)
At the start: 60 parts, among them IC901 BME680, J1 Conn_ARM_JTAG_SWD_10, J2 Conn_01x01_Pin, J3 Conn_01x01_Pin, SW1 SW_Push, U1 nRF52840, U2 HDC2080, U3 SM351LT, U4 TPS610981, U5 OPT3001, Y1 32MHz, Y2 32.768kHz

Commit message: Layout done
Parts:
- removed D1, D2: LED, LED_SMD:LED_0603_1608Metric, symbol Device:LED
- removed SW1: SW_Push, Button_Switch_SMD:SW_SPST_B3U-1000P-B, symbol Switch:SW_Push
- added LED101, LED501: G, LED:LED0603, symbol LED:LED
- added SW401: KMR231GLFS, Switches:TACT_SW4_KMR2, symbol Switches:TACT_SW4
- C11, C18, C23: footprint Capacitor_SMD:C_0603_1608Metric -> Passives:C0603
- L1: value 4.7nH -> 4.7n
- R1, R7: value 0R -> 0
- R2, R8: value 330R -> 330
- R4: value 402R -> 402; footprint Resistor_SMD:R_0603_1608Metric -> Passives:R0603
- R5, R6: value 10K -> 10k
- Y1: value 32MHz -> ABM8W-32.0000MHZ-8-B1U-T3
- Y2: value 32.768kHz -> Q13FC13500004
Connections:
- net GND: now also SW401.1A, SW401.1B
- net LED1: now also LED101.A
- net LED2: now also LED501.A
- net SW1: now also SW401.2A, SW401.2B
- net at R8.2: now also LED501.C
- net at R2.2: now also LED101.C

Commit message: Populated
Parts:
- SW401: value KMR231GLFS -> KMR211NGLFS
- U1: value nRF52840 -> NRF52840-QIAA-R
Connections:
- no-connect marks 9 -> 46
Other:
- moved on the sheet: C1, C10, C101, C11, C12, C13, C14, C15, C16, C17, C2, C3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
