File: PCB/Zicada Board/Zicada.kicad_pcb (KiCad board)
At the start: 4 copper layers, 57.4 x 12 mm, 63 parts, among them IC901 BME680, J1 Conn_ARM_JTAG_SWD_10, J2 Conn_01x01_Pin, J3 Conn_01x01_Pin, SW1 SW_Push, U1 nRF52840, U2 HDC2080, U3 SM351LT, U4 TPS610981, U5 OPT3001, Y1 32MHz, Y2 32.768kHz

Commit message: Layout done
Parts:
- removed D1, D2: LED, LED_SMD:LED_0603_1608Metric
- removed SW1: SW_Push, Button_Switch_SMD:SW_SPST_B3U-1000P-B
- added LED101: G, LED:LED0603, F.Cu at (171.2, 93.0)
- added LED501: G, LED:LED0603, F.Cu at (139.2, 92.8)
- added SW401: KMR231GLFS, Switches:TACT_SW4_KMR2, F.Cu at (141.5, 93.0)
- C11, C18, C23: footprint Capacitor_SMD:C_0603_1608Metric -> Passives:C0603
- L1: value 4.7nH -> 4.7n
- R1, R7: value 0R -> 0
- R2, R8: value 330R -> 330
- R4: value 402R -> 402; footprint Resistor_SMD:R_0603_1608Metric -> Passives:R0603
- R5, R6: value 10K -> 10k
- Y1: value 32MHz -> ABM8W-32.0000MHZ-8-B1U-T3
- Y2: value 32.768kHz -> Q13FC13500004
Routing:
- net /SW1: track 16.8 -> 20.3 mm
- net GND: vias 81 -> 82

Commit message: Populated
Parts:
- SW401: value KMR231GLFS -> KMR211NGLFS
- U1: value nRF52840 -> NRF52840-QIAA-R
